Commit message: 2

File: rm_simulation/livox_laser_simulation_RO2/urdf/mid360.xacro (robot description, xacro)
@@ -24,5 +24,5 @@
         <origin xyz="0.025 -0.0265 -0.025" rpy="${pi/2} 0 ${pi}"/>
         <geometry>
-          <mesh filename="model://mid360.stl" scale="0.0008 0.0008 0.0008"/>
+          <mesh filename="package://pb_rm_simulation/meshes/mid360.stl" scale="0.0008 0.0008 0.0008"/>
         </geometry>
       </visual>
